Commit message: pushing for safety. Added wheels, rolling, issues with non swing legs swinging anyway

File: legged_examples/legged_unitree/legged_unitree_description/urdf/common/leg.xacro (robot description, xacro)
@@ -157,4 +157,59 @@
             </inertial>
         </link>
+        <joint name="${prefix}_switcher" type="prismatic">
+            <origin rpy="${pi/2.0} 0.5 0" xyz="0.02 0 0.05"/>
+            <parent link="${prefix}_FOOT"/>
+            <child link="${prefix}_dummy"/>
+            <axis xyz="0 1 0"/>
+            <dynamics damping="0." friction="0"/>
+            <limit effort="1e100" velocity="5" lower="-0.05" upper="0.05"/>
+        </joint>
+        <link name="${prefix}_dummy">
+            <inertial>
+                <origin rpy="0 0 0" xyz="0 0 0"/>
+                <mass value="0.001"/>
+                <inertia
+                        ixx="0.000001696" ixy="0" ixz="0"
+                        iyy="0.000001696" iyz="0"
+                        izz="0.000003226"/>
+            </inertial>
+        </link>
+        <joint name="${prefix}_roller" type="revolute">
+            <origin rpy="0 0 0" xyz="0 0 0"/>
+            <parent link="${prefix}_dummy"/>
+            <child link="${prefix}_wheel"/>
+            <axis xyz="0 0 1"/>
+            <dynamics damping="0" friction="0.03"/>
+            <limit effort="0" velocity="10" lower="-1e100" upper="1e100"/>
+        </joint>
+        <link name="${prefix}_wheel">
+            <visual>
+                <origin rpy="0 0 0" xyz="0 0 0"/>
+                <geometry>
+                    <cylinder length="0.01" radius="0.03"/>
+                </geometry>
+                <material name="orange"/>
+            </visual>
+            <visual>
+                <geometry>
+                    <mesh filename="${mesh_path}/wheel.dae" />
+                </geometry>
+                <material name=""/>
+            </visual>
+            <collision>
+                <origin rpy="0 0 0" xyz="0 0 0"/>
+                <geometry>
+                    <cylinder length="0.01" radius="0.03"/>
+                </geometry>
+            </collision>
+            <inertial>
+                <origin rpy="0 0 0" xyz="0 0 0"/>
+                <mass value="0.025"/>
+                <inertia
+                        ixx="0.00001696" ixy="0" ixz="0"
+                        iyy="0.00001696" iyz="0"
+                        izz="0.00003226"/>
+            </inertial>
+        </link>
         <gazebo reference="${prefix}_foot_fixed">
             <disableFixedJointLumping>true</disableFixedJointLumping>
@@ -181,9 +236,25 @@
             <mu1>0.6</mu1>
             <mu2>0.6</mu2>
-            <self_collide>1</self_collide>
+            <self_collide>0</self_collide>
             <material>Gazebo/DarkGrey</material>
             <kp value="1000000.0"/>
             <kd value="100.0"/>
         </gazebo>
+        <gazebo reference="${prefix}_wheel">
+            <self_collide>false</self_collide>
+            <mu1>0.6</mu1>
+            <mu2>0.6</mu2>
+            <kp value="1000000.0"/>
+            <kd value="100.0"/>
+        </gazebo>
+        <gazebo reference="${prefix}_switcher">
+            <provide_feedback>true</provide_feedback>
+            <kp>500000.0</kp>
+            <kd>1000.0</kd>
+            <fudge_factor>0.0001</fudge_factor>
+            <cfm>0.0</cfm>
+            <erp>0.2</erp>
+            <bounce>0.0</bounce>
+        </gazebo>
         <xacro:leg_transmission name="${prefix}"/>
     </xacro:macro>

File: legged_examples/legged_unitree/legged_unitree_description/urdf/common/materials.xacro (robot description, xacro)
@@ -9,4 +9,9 @@
     <material name="green">
         <color rgba="0.0 0.8 0.0 1.0"/>
+    </material>
+    <material name="wheelTexture">
+        <script>
+            <uri>wheelTexture.material</uri>
+        </script>
     </material>
     <material name="grey">

File: legged_examples/legged_unitree/legged_unitree_description/urdf/common/transmission.xacro (robot description, xacro)
@@ -32,4 +32,24 @@
             </actuator>
         </transmission>
+        <transmission name="${prefix}_switcher_tran">
+            <type>transmission_interface/SimpleTransmission</type>
+            <joint name="${prefix}_switcher">
+                <hardwareInterface>hardware_interface/EffortJointInterface</hardwareInterface>
+            </joint>
+            <actuator name="${prefix}_switcher_motor">
+                <hardwareInterface>hardware_interface/EffortJointInterface</hardwareInterface>
+                <mechanicalReduction>1</mechanicalReduction>
+            </actuator>
+        </transmission>
+        <transmission name="${prefix}_roller_tran">
+            <type>transmission_interface/SimpleTransmission</type>
+            <joint name="${prefix}_roller">
+                <hardwareInterface>hardware_interface/EffortJointInterface</hardwareInterface>
+            </joint>
+            <actuator name="${prefix}_roller_motor">
+                <hardwareInterface>hardware_interface/EffortJointInterface</hardwareInterface>
+                <mechanicalReduction>1</mechanicalReduction>
+            </actuator>
+        </transmission>
     </xacro:macro>
 </robot>

Commit message: it's rolling now

File: legged_examples/legged_unitree/legged_unitree_description/urdf/common/leg.xacro (robot description, xacro)
@@ -163,5 +163,5 @@
             <axis xyz="0 1 0"/>
             <dynamics damping="0." friction="0"/>
-            <limit effort="1e100" velocity="5" lower="-0.05" upper="0.05"/>
+            <limit effort="1e100" velocity="10" lower="-0.05" upper="0.05"/>
         </joint>
         <link name="${prefix}_dummy">
@@ -175,20 +175,13 @@
             </inertial>
         </link>
-        <joint name="${prefix}_roller" type="revolute">
+        <joint name="${prefix}_roller" type="continuous">
             <origin rpy="0 0 0" xyz="0 0 0"/>
             <parent link="${prefix}_dummy"/>
             <child link="${prefix}_wheel"/>
             <axis xyz="0 0 1"/>
-            <dynamics damping="0" friction="0.03"/>
-            <limit effort="0" velocity="10" lower="-1e100" upper="1e100"/>
+            <dynamics damping="0.00" friction="0.00"/>
+            <limit effort="0" velocity="10"/>
         </joint>
         <link name="${prefix}_wheel">
-            <visual>
-                <origin rpy="0 0 0" xyz="0 0 0"/>
-                <geometry>
-                    <cylinder length="0.01" radius="0.03"/>
-                </geometry>
-                <material name="orange"/>
-            </visual>
             <visual>
                 <geometry>
@@ -243,8 +236,19 @@
         <gazebo reference="${prefix}_wheel">
             <self_collide>false</self_collide>
-            <mu1>0.6</mu1>
-            <mu2>0.6</mu2>
-            <kp value="1000000.0"/>
-            <kd value="100.0"/>
+            <fdir1>0 0 1</fdir1>  <!-- forces friction to against rolling direction-->
+            <!-- Friction: low in rolling dir (mu1), higher sideways (mu2) -->
+            <mu1>100.00</mu1>
+            <mu2>0.03</mu2>
+            <!-- Allow a bit of micro-slip to avoid stiction -->
+            <slip1>0.00</slip1>
+            <slip2>0.00</slip2>
+            <!-- Soften contact to avoid impulsive locking -->
+            <kp>200000.0</kp>   <!-- 2e5 -->
+            <kd>20.0</kd>
+            <!-- increase allowed interpenetration before big forces -->
+            <min_depth>0.002</min_depth>
+        </gazebo>
+        <gazebo reference="${prefix}_roller">
+            <passive>true</passive>
         </gazebo>
         <gazebo reference="${prefix}_switcher">

Commit message: rolling well now. Adding terrain next

File: legged_examples/legged_unitree/legged_unitree_description/urdf/common/leg.xacro (robot description, xacro)
@@ -158,10 +158,10 @@
         </link>
         <joint name="${prefix}_switcher" type="prismatic">
-            <origin rpy="${pi/2.0} 0.5 0" xyz="0.02 0 0.05"/>
+            <origin rpy="0 0.5 0" xyz="0.02 0 0.05"/>
             <parent link="${prefix}_FOOT"/>
             <child link="${prefix}_dummy"/>
-            <axis xyz="0 1 0"/>
-            <dynamics damping="0." friction="0"/>
-            <limit effort="1e100" velocity="10" lower="-0.05" upper="0.05"/>
+            <axis xyz="0 0 1"/>
+            <dynamics damping="10.0" friction="0.5"/>
+            <limit effort="1e100" velocity="10" lower="-0.045" upper="0.05"/>
         </joint>
         <link name="${prefix}_dummy">
@@ -176,5 +176,5 @@
         </link>
         <joint name="${prefix}_roller" type="continuous">
-            <origin rpy="0 0 0" xyz="0 0 0"/>
+            <origin rpy="${pi/2.0} 0 0" xyz="0 0 0"/>
             <parent link="${prefix}_dummy"/>
             <child link="${prefix}_wheel"/>
@@ -193,5 +193,5 @@
                 <origin rpy="0 0 0" xyz="0 0 0"/>
                 <geometry>
-                    <cylinder length="0.01" radius="0.03"/>
+                    <cylinder length="0.02" radius="0.03"/>
                 </geometry>
             </collision>
@@ -234,29 +234,31 @@
             <kd value="100.0"/>
         </gazebo>
-        <gazebo reference="${prefix}_wheel">
-            <self_collide>false</self_collide>
-            <fdir1>0 0 1</fdir1>  <!-- forces friction to against rolling direction-->
-            <!-- Friction: low in rolling dir (mu1), higher sideways (mu2) -->
-            <mu1>100.00</mu1>
-            <mu2>0.03</mu2>
-            <!-- Allow a bit of micro-slip to avoid stiction -->
-            <slip1>0.00</slip1>
-            <slip2>0.00</slip2>
-            <!-- Soften contact to avoid impulsive locking -->
-            <kp>200000.0</kp>   <!-- 2e5 -->
-            <kd>20.0</kd>
-            <!-- increase allowed interpenetration before big forces -->
-            <min_depth>0.002</min_depth>
-        </gazebo>
         <gazebo reference="${prefix}_roller">
             <passive>true</passive>
         </gazebo>
+        <gazebo reference="${prefix}_wheel">
+            <!-- <wheel_slip>
+                <slip_compliance_lateral>0.0</slip_compliance_lateral>
+                <slip_compliance_longitudinal>0.0</slip_compliance_longitudinal>
+                <wheel_normal_force>1000</wheel_normal_force>
+            </wheel_slip> -->
+            <self_collide>false</self_collide>
+            <fdir1>1 0 0</fdir1>  <!-- forces friction to against rolling direction-->
+            <!-- Friction: low in rolling dir (mu1), higher sideways (mu2) -->
+            <mu1>0.02</mu1>
+            <mu2>5.0</mu2>
+            <slip1>0.01</slip1>
+            <slip2>0.00</slip2>
+            <min_depth>0.01</min_depth>
+            <kp>100000.0</kp>
+            <kd>450.0</kd>
+        </gazebo>
         <gazebo reference="${prefix}_switcher">
             <provide_feedback>true</provide_feedback>
-            <kp>500000.0</kp>
-            <kd>1000.0</kd>
+            <kp>50000.0</kp>
+            <kd>10000.0</kd>
             <fudge_factor>0.0001</fudge_factor>
-            <cfm>0.0</cfm>
-            <erp>0.2</erp>
+            <cfm>1e-9</cfm>
+            <erp>0.8</erp>
             <bounce>0.0</bounce>
         </gazebo>
